Commit message: add camera to the sequential_testbed

File: urdf/accessories.urdf.xacro (robot description, xacro)
@@ -45,4 +45,7 @@
       <child link="$(optenv JACKAL_NAVSAT_MOUNT rear)_navsat" />
     </joint>
+  </xacro:if>
+  <xacro:if value="$(optenv CAMERA 0)">
+    <xacro:include filename="$(find jackal_helper)/urdf/accessories/camera.urdf.xacro" />
   </xacro:if>
   <!-- Common camera mounts and accessory URDFs. -->

File: urdf/accessories/VLP-16.urdf.xacro (robot description, xacro)
@@ -9,5 +9,8 @@
     </joint>
     <link name="${name}_base_link">
-      <inertial>
+      <inertial>      <VLP-16 parent="$(optenv JACKAL_LASER_MOUNT front)_mount"
+              name="front_laser">
+        <origin xyz="0 0 0" rpy="0 0 0" />
+      </VLP-16>
         <mass value="0.83"/>
         <origin xyz="0 0 0.03585"/>
